Commit message: Fork for CTU husky

File: husky_description/urdf/empty.urdf (robot description, URDF)
Before this commit: robot None, 0 links, 0 joints
Links:
- added link laser_base
- added link lidar
- added link rs_lidar
- added link rslidar
Joints:
- added joint laser_base_joint: type fixed, parent base_link, child laser_base, origin xyz=0 0 0.4 rpy=0 0 0
- added joint lidar_centre_joint: type fixed, parent rs_lidar, child lidar, origin xyz=0 0 0.04536 rpy=0 0 0
- added joint rs_lidar_centre_joint: type fixed, parent rs_lidar, child rslidar, origin xyz=0 0 0.04536 rpy=0 0 0
- added joint rs_lidar_joint: type fixed, parent laser_base, child rs_lidar, origin xyz=0 0 0 rpy=0 0 0

Commit message: transformations of final build added, camera tf prepared

File: husky_description/urdf/empty.urdf (robot description, URDF)
Before this commit: robot None, 4 links, 4 joints
Links:
- removed link laser_base
- added link cam1_base
- added link cam2_base
- added link mount_base
Joints:
- removed joint laser_base_joint
- added joint cam1_base_joint: type fixed, parent mount_base, child cam1_base, origin xyz=0.0502 0.0365 -0.006 rpy=0.942478 -1.5708 3.1416
- added joint cam2_base_joint: type fixed, parent mount_base, child cam2_base, origin xyz=0.0502 -0.0365 -0.006 rpy=5.34071 -1.5708 3.1416
- added joint mount_base_joint: type fixed, parent base_link, child mount_base, origin xyz=0 -0.01 0.395 rpy=0 0 0
- joint rs_lidar_joint: origin xyz=0 0 0 rpy=0 0 0 -> xyz=0 0 0.1 rpy=0 0 0; parent laser_base -> mount_base
